Commit message: update DH2URDF

File: uthai_utils/DH2URDF/myRobot.xacro (robot description, xacro)
@@ -1 +1,61 @@
-<robot name="myRobot" xmlns:xacro="http://www.ros.org/wiki/xacro"><!--Uthai Humanoid, FIBO, KMUTT, Thailand, 2017--><!--This file generated by Liews Wuttipat--><macro name="DH_fixed" params="parent child xyz rpy"><joint name="jd_${child}" type="fixed"><parent link="fd_${parent}" /><child link="f_${child}" /><origin rpy="${rpy}" xyz="${xyz}" /></joint><link name="f_${child}" /><link name="fd_${child}" /></macro><macro name="DH_F" params="parent child xyz rpy id"><DH_fixed child="${child}" parent="${parent}" rpy="${rpy}" xyz="${xyz}" /><joint name="jf_${id}" type="fixed"><parent link="f_${child}" /><child link="fd_${child}" /></joint></macro><macro name="DH_R" params="parent child xyz rpy id"><DH_fixed child="${child}" parent="${parent}" rpy="${rpy}" xyz="${xyz}" /><joint name="j_${id}" type="revolute"><parent link="f_${child}" /><child link="fd_${child}" /><axis xyz="0 0 1" /><limit effort="10" lower="-2.6179939" upper="2.6179939" velocity="5.6548668" /></joint></macro><!--End Macro to make dummy link--><link name="base_link" /><link name="fd_base_link" /><joint name="fixed_fd" type="fixed"><parent link="base_link" /><child link="fd_base_link" /></joint><DH_R child="0" id="1" parent="base_link" rpy="0.0 -0.0 -1.5707963267948966" xyz="5.51091059616e-18 -0.09 -0.055" /><DH_R child="1" id="2" parent="0" rpy="-1.5707963267948966 -0.0 1.5707963267948966" xyz="0.0 0.0 -0.04" /><DH_R child="2" id="3" parent="1" rpy="1.5707963267948966 -0.0 1.5707963267948966" xyz="0.0 0.0 0.0" /><DH_R child="3" id="4" parent="2" rpy="-1.5707963267948966 -0.0 0.0" xyz="0.3 0.0 0.0" /><DH_R child="4" id="5" parent="3" rpy="0.0 -0.0 0.0" xyz="0.315 0.0 0.0" /><DH_R child="5" id="6" parent="4" rpy="1.5707963267948966 -0.0 0.0" xyz="0.0 0.0 0.0" /><DH_F child="6" id="1" parent="5" rpy="-1.5707963267948966 -0.0 0.0" xyz="0.045 0.0 0.0" /><DH_F child="7" id="2" parent="6" rpy="1.5707963267948966 -0.0 -1.5707963267948966" xyz="3.55147571753e-18 -0.058 0.0" /><DH_R child="10" id="7" parent="base_link" rpy="0.0 -0.0 1.5707963267948966" xyz="5.51091059616e-18 0.09 -0.055" /><DH_R child="11" id="8" parent="10" rpy="-1.5707963267948966 -0.0 -1.5707963267948966" xyz="0.0 -0.0 -0.04" /><DH_R child="12" id="9" parent="11" rpy="1.5707963267948966 -0.0 1.5707963267948966" xyz="0.0 0.0 0.0" /><DH_R child="13" id="10" parent="12" rpy="-1.5707963267948966 -0.0 0.0" xyz="0.3 0.0 0.0" /><DH_R child="14" id="11" parent="13" rpy="0.0 -0.0 0.0" xyz="0.315 0.0 0.0" /><DH_R child="15" id="12" parent="14" rpy="1.5707963267948966 -0.0 0.0" xyz="0.0 0.0 0.0" /><DH_F child="16" id="3" parent="15" rpy="-1.5707963267948966 -0.0 0.0" xyz="0.045 0.0 0.0" /><DH_F child="17" id="4" parent="16" rpy="1.5707963267948966 -0.0 -1.5707963267948966" xyz="3.55147571753e-18 -0.058 0.0" /><DH_F child="20" id="5" parent="base_link" rpy="0.0 -0.0 0.0" xyz="0.0 0.0 0.29" /><DH_R child="21" id="13" parent="20" rpy="-1.5707963267948966 -0.0 0.0" xyz="0.0 0.0 0.0" /><DH_F child="22" id="6" parent="21" rpy="1.5707963267948966 -0.0 1.5707963267948966" xyz="0.0 0.0 -0.145" /><DH_F child="23" id="7" parent="22" rpy="0.0 -0.0 0.0" xyz="0.32 0.0 0.0" /><DH_F child="30" id="8" parent="base_link" rpy="0.0 -0.0 0.0" xyz="0.0 0.0 0.29" /><DH_R child="31" id="14" parent="30" rpy="1.5707963267948966 -0.0 0.0" xyz="0.0 0.0 0.0" /><DH_F child="32" id="9" parent="31" rpy="-1.5707963267948966 -0.0 -1.5707963267948966" xyz="0.0 -0.0 -0.145" /><DH_F child="33" id="10" parent="32" rpy="0.0 -0.0 0.0" xyz="0.32 0.0 0.0" /></robot>
+<robot name="myRobot"
+    xmlns:xacro="http://www.ros.org/wiki/xacro">
+    <!--Uthai Humanoid, FIBO, KMUTT, Thailand, 2017-->
+    <!--This file generated by Liews Wuttipat-->
+    <macro name="DH_fixed" params="parent child xyz rpy">
+        <joint name="jd_${child}" type="fixed">
+            <parent link="fd_${parent}" />
+            <child link="f_${child}" />
+            <origin rpy="${rpy}" xyz="${xyz}" />
+        </joint>
+        <link name="f_${child}" />
+        <link name="fd_${child}" />
+    </macro>
+    <macro name="DH_F" params="parent child xyz rpy id">
+        <DH_fixed child="${child}" parent="${parent}" rpy="${rpy}" xyz="${xyz}" />
+        <joint name="jf_${id}" type="fixed">
+            <parent link="f_${child}" />
+            <child link="fd_${child}" />
+        </joint>
+    </macro>
+    <macro name="DH_R" params="parent child xyz rpy id">
+        <DH_fixed child="${child}" parent="${parent}" rpy="${rpy}" xyz="${xyz}" />
+        <joint name="j_${id}" type="revolute">
+            <parent link="f_${child}" />
+            <child link="fd_${child}" />
+            <axis xyz="0 0 1" />
+            <limit effort="10" lower="-2.6179939" upper="2.6179939" velocity="5.6548668" />
+        </joint>
+    </macro>
+    <!--End Macro to make dummy link-->
+    <link name="base_link" />
+    <link name="fd_base_link" />
+    <joint name="fixed_fd" type="fixed">
+        <parent link="base_link" />
+        <child link="fd_base_link" />
+    </joint>
+    <DH_R child="0" id="1" parent="base_link" rpy="0.0 -0.0 -1.5707963267948966" xyz="5.51091059616e-18 -0.09 -0.055" />
+    <DH_R child="1" id="2" parent="0" rpy="-1.5707963267948966 -0.0 1.5707963267948966" xyz="0.0 0.0 -0.04" />
+    <DH_R child="2" id="3" parent="1" rpy="1.5707963267948966 -0.0 1.5707963267948966" xyz="0.0 0.0 0.0" />
+    <DH_R child="3" id="4" parent="2" rpy="-1.5707963267948966 -0.0 0.0" xyz="0.3 0.0 0.0" />
+    <DH_R child="4" id="5" parent="3" rpy="0.0 -0.0 0.0" xyz="0.315 0.0 0.0" />
+    <DH_R child="5" id="6" parent="4" rpy="1.5707963267948966 -0.0 0.0" xyz="0.0 0.0 0.0" />
+    <DH_F child="6" id="1" parent="5" rpy="-1.5707963267948966 -0.0 0.0" xyz="0.045 0.0 0.0" />
+    <DH_F child="7" id="2" parent="6" rpy="1.5707963267948966 -0.0 -1.5707963267948966" xyz="3.55147571753e-18 -0.058 0.0" />
+    <DH_R child="10" id="7" parent="base_link" rpy="0.0 -0.0 1.5707963267948966" xyz="5.51091059616e-18 0.09 -0.055" />
+    <DH_R child="11" id="8" parent="10" rpy="-1.5707963267948966 -0.0 -1.5707963267948966" xyz="0.0 -0.0 -0.04" />
+    <DH_R child="12" id="9" parent="11" rpy="1.5707963267948966 -0.0 1.5707963267948966" xyz="0.0 0.0 0.0" />
+    <DH_R child="13" id="10" parent="12" rpy="-1.5707963267948966 -0.0 0.0" xyz="0.3 0.0 0.0" />
+    <DH_R child="14" id="11" parent="13" rpy="0.0 -0.0 0.0" xyz="0.315 0.0 0.0" />
+    <DH_R child="15" id="12" parent="14" rpy="1.5707963267948966 -0.0 0.0" xyz="0.0 0.0 0.0" />
+    <DH_F child="16" id="3" parent="15" rpy="-1.5707963267948966 -0.0 0.0" xyz="0.045 0.0 0.0" />
+    <DH_F child="17" id="4" parent="16" rpy="1.5707963267948966 -0.0 -1.5707963267948966" xyz="3.55147571753e-18 -0.058 0.0" />
+    <DH_F child="20" id="5" parent="base_link" rpy="0.0 -0.0 0.0" xyz="0.0 0.0 0.29" />
+    <DH_R child="21" id="13" parent="20" rpy="-1.5707963267948966 -0.0 0.0" xyz="0.0 0.0 0.0" />
+    <DH_F child="22" id="6" parent="21" rpy="1.5707963267948966 -0.0 1.5707963267948966" xyz="0.0 0.0 -0.145" />
+    <DH_F child="23" id="7" parent="22" rpy="0.0 -0.0 0.0" xyz="0.32 0.0 0.0" />
+    <DH_F child="30" id="8" parent="base_link" rpy="0.0 -0.0 0.0" xyz="0.0 0.0 0.29" />
+    <DH_R child="31" id="14" parent="30" rpy="-1.5707963267948966 -0.0 0.0" xyz="0.0 0.0 0.0" />
+    <DH_F child="32" id="9" parent="31" rpy="-1.5707963267948966 -0.0 -1.5707963267948966" xyz="0.0 -0.0 -0.145" />
+    <DH_F child="33" id="10" parent="32" rpy="0.0 -0.0 0.0" xyz="0.32 0.0 0.0" />
+</robot>
